File: CurrentSinkOrSwim.sch (KiCad schematic (older format))
At the start: 0 parts

Commit message: Initial schematic
Parts:
- added C? (x2): C, ~, symbol C
- added P?: CONN_2, symbol CONN_2
- added Q?: MOSFET_N, ~, symbol MOSFET_N
- added R? (x2): R, ~, symbol R
- added RV?: POT, ~, symbol POT
- added U? (x2): LMV358, ~, symbol LMV358
- added U?: TC1016, ~, symbol TC1016
Connections:
- net labels added: GND
- wire segments 0 -> 23
Changed lines of the file:
@@
 LIBS:contrib
 LIBS:valves
+LIBS:CurrentSinkOrSwim
 EELAYER 27 0
 EELAYER END
@@
 Sheet 1 1
 Title ""
-Date "28 jun 2015"
+Date "2 jul 2015"
 Rev ""
 Comp ""
@@
 Comment4 ""
 $EndDescr
+$Comp
+L LMV358 U?
+U 1 1 5594980D
+P 2650 2200
+F 0 "U?" H 2600 2400 60  0000 L CNN
+F 1 "LMV358" H 2600 1950 60  0000 L CNN
+F 2 "~" H 2650 2200 60  0000 C CNN
+F 3 "~" H 2650 2200 60  0000 C CNN
+	1    2650 2200
+	1    0    0    -1
+$EndComp
+$Comp
+L R R?
+U 1 1 55949826
+P 4150 3450
+F 0 "R?" V 4230 3450 40  0000 C CNN
+F 1 "R" V 4157 3451 40  0000 C CNN
+F 2 "~" V 4080 3450 30  0000 C CNN
+F 3 "~" H 4150 3450 30  0000 C CNN
+	1    4150 3450
+	1    0    0    1
+$EndComp
+$Comp
+L R R?
+U 1 1 55949844
+P 1350 3600
+F 0 "R?" V 1430 3600 40  0000 C CNN
+F 1 "R" V 1357 3601 40  0000 C CNN
+F 2 "~" V 1280 3600 30  0000 C CNN
+F 3 "~" H 1350 3600 30  0000 C CNN
+	1    1350 3600
+	1    0    0    -1
+$EndComp
+$Comp
+L MOSFET_N Q?
+U 1 1 55949853
+P 4050 2200
+F 0 "Q?" H 4060 2370 60  0000 R CNN
+F 1 "MOSFET_N" H 4060 2050 60  0000 R CNN
+F 2 "~" H 4050 2200 60  0000 C CNN
+F 3 "~" H 4050 2200 60  0000 C CNN
+	1    4050 2200
+	1    0    0    -1
+$EndComp
+$Comp
+L GND #PWR?
+U 1 1 55949876
+P 4150 4250
+F 0 "#PWR?" H 4150 4250 30  0001 C CNN
+F 1 "GND" H 4150 4180 30  0001 C CNN
+F 2 "" H 4150 4250 60  0000 C CNN
+F 3 "" H 4150 4250 60  0000 C CNN
+	1    4150 4250
+	1    0    0    -1
+$EndComp
+$Comp
+L GND #PWR?
+U 1 1 55949885
+P 2550 2700
+F 0 "#PWR?" H 2550 2700 30  0001 C CNN
+F 1 "GND" H 2550 2630 30  0001 C CNN
+F 2 "" H 2550 2700 60  0000 C CNN
+F 3 "" H 2550 2700 60  0000 C CNN
+	1    2550 2700
+	1    0    0    -1
+$EndComp
+$Comp
+L TC1016 U?
+U 1 1 55949CB6
+P 3300 1200
+F 0 "U?" H 3450 1004 60  0000 C CNN
+F 1 "TC1016" H 3300 1400 60  0000 C CNN
+F 2 "~" H 3300 1200 60  0000 C CNN
+F 3 "~" H 3300 1200 60  0000 C CNN
+	1    3300 1200
+	-1   0    0    -1
+$EndComp
+$Comp
+L GND #PWR?
+U 1 1 55949CD9
+P 3300 1950
+F 0 "#PWR?" H 3300 1950 30  0001 C CNN
+F 1 "GND" H 3300 1880 30  0001 C CNN
+F 2 "" H 3300 1950 60  0000 C CNN
+F 3 "" H 3300 1950 60  0000 C CNN
+	1    3300 1950
+	1    0    0    -1
+$EndComp
+$Comp
+L C C?
+U 1 1 55949E34
+P 3800 1450
+F 0 "C?" H 3800 1550 40  0000 L CNN
+F 1 "C" H 3806 1365 40  0000 L CNN
+F 2 "~" H 3838 1300 30  0000 C CNN
+F 3 "~" H 3800 1450 60  0000 C CNN
+	1    3800 1450
+	1    0    0    -1
+$EndComp
+$Comp
+L C C?
+U 1 1 55949E43
+P 2800 1450
+F 0 "C?" H 2800 1550 40  0000 L CNN
+F 1 "C" H 2806 1365 40  0000 L CNN
+F 2 "~" H 2838 1300 30  0000 C CNN
+F 3 "~" H 2800 1450 60  0000 C CNN
+	1    2800 1450
+	1    0    0    -1
+$EndComp
+Wire Wire Line
+	2550 2700 2550 2600
+Wire Wire Line
+	4150 2400 4150 3200
+Wire Wire Line
+	3850 2200 3150 2200
+Wire Wire Line
+	1500 1150 1500 2450
+Wire Wire Line
+	2550 1150 2550 1800
+Wire Wire Line
+	1350 2700 1350 3350
+Wire Wire Line
+	4150 3700 4150 4250
+Wire Wire Line
+	2150 2100 1800 2100
+Wire Wire Line
+	1800 2100 1800 3000
+Wire Wire Line
+	1800 3000 1350 3000
+Connection ~ 1350 3000
+Wire Wire Line
+	2150 2300 2150 3000
+Wire Wire Line
+	2150 3000 4150 3000
+Connection ~ 4150 3000
+Wire Wire Line
+	3300 1950 3300 1450
+Connection ~ 2550 1150
+Wire Wire Line
+	3700 1150 4150 1150
+Wire Wire Line
+	4150 900  4150 2000
+Wire Wire Line
+	4150 900  5100 900
+Connection ~ 4150 1150
+Wire Wire Line
+	2800 1300 2800 1150
+Connection ~ 2800 1150
+Wire Wire Line
+	2800 1650 3800 1650
+Connection ~ 3300 1650
+Wire Wire Line
+	3800 1250 3800 1150
+Connection ~ 3800 1150
+$Comp
+L POT RV?
+U 1 1 55949F38
+P 1350 2450
+F 0 "RV?" H 1350 2350 50  0000 C CNN
+F 1 "POT" H 1350 2450 50  0000 C CNN
+F 2 "~" H 1350 2450 60  0000 C CNN
+F 3 "~" H 1350 2450 60  0000 C CNN
+	1    1350 2450
+	0    1    1    0
+$EndComp
+Wire Wire Line
+	1500 1150 2900 1150
+Wire Wire Line
+	1350 3850 4150 3850
+Connection ~ 4150 3850
+$Comp
+L CONN_2 P?
+U 1 1 5594A019
+P 5450 1000
+F 0 "P?" V 5400 1000 40  0000 C CNN
+F 1 "CONN_2" V 5500 1000 40  0000 C CNN
+F 2 "" H 5450 1000 60  0000 C CNN
+F 3 "" H 5450 1000 60  0000 C CNN
+	1    5450 1000
+	1    0    0    -1
+$EndComp
+$Comp
+L GND #PWR?
+U 1 1 5594A04E
+P 5000 1250
+F 0 "#PWR?" H 5000 1250 30  0001 C CNN
+F 1 "GND" H 5000 1180 30  0001 C CNN
+F 2 "" H 5000 1250 60  0000 C CNN
+F 3 "" H 5000 1250 60  0000 C CNN
+	1    5000 1250
+	1    0    0    -1
+$EndComp
+Wire Wire Line
+	5100 1100 5000 1100
+Wire Wire Line
+	5000 1100 5000 1250
+$Comp
+L LMV358 U?
+U 2 1 5594A0E3
+P 5750 3100
+F 0 "U?" H 5700 3300 60  0000 L CNN
+F 1 "LMV358" H 5700 2850 60  0000 L CNN
+F 2 "~" H 5750 3100 60  0000 C CNN
+F 3 "~" H 5750 3100 60  0000 C CNN
+	2    5750 3100
+	1    0    0    -1
+$EndComp
 $EndSCHEMATC
